Commit message: Mostly comment removals

File: turtlex/turtlex_description/robots/rgbd.urdf.xacro (robot description, xacro)
@@ -2,15 +2,6 @@
 <robot name="rgbd" xmlns:xacro="http://www.ros.org/wiki/xacro">
 <xacro:macro name="rgbd_main" params="parent">
-	<!--<xacro:include filename="$(find turtlex_description)/urdf/common_properties.urdf.xacro"/>-->
 	<!-- 3D sensor -->
 	<xacro:include filename="$(find turtlex_description)/urdf/asus_xtion_pro.urdf.xacro"/>
-	<!--<link name="rgbd_base_link">
-		<visual>
-			<origin xyz="0 0 0" rpy="0 0 0"/>
-			<geometry>
-				<box size="0.001 0.001 0.001" />
-			</geometry>
-		</visual>
-	</link>-->
 	<xacro:sensor_asus_xtion_pro parent="${parent}"/>
 </xacro:macro>

File: turtlex/turtlex_description/robots/widowx_arm.urdf.xacro (robot description, xacro)
@@ -3,18 +3,6 @@
 <xacro:macro name="widowx_arm_main" params="parent">
 	<xacro:include filename="$(find turtlex_description)/urdf/widowx.urdf.xacro"/>
-	<!--<link name="widow_base_footprint">
-		<visual>
-			<origin xyz="0 0 0" rpy="0 0 0"/>
-			<geometry>
-				<box size="0.001 0.001 0.001" />
-			</geometry>
-		</visual>
-	</link>
-	<joint name="fixed" type="fixed">
-    	<parent link="${parent}"/>
-    	<child link="widow_base_footprint"/>
- 	</joint>-->
 	<xacro:widowx_arm parent="${parent}">
-		<!-- moving it a bit backwards in order to leave some space for the laser sensors on the front-->
+		<!-- moving the arm a bit backwards in order to leave some space for the laser sensors on the front -->
 		<origin xyz="-0.007 0.0 0.0" rpy="0.0 0.0 0.0"/>
 	</xacro:widowx_arm>

File: turtlex/turtlex_description/urdf/asus_xtion_pro.urdf.xacro (robot description, xacro)
@@ -1,9 +1,6 @@
-<?xml version="1.0" encoding="utf-8"?> <!-- NOTA BENE: questa e la asus xtion pro LIVE (quella non live non ha rgb) -->
-<robot name="sensor_asus_xtion_pro" xmlns:xacro="http://www.ros.org/wiki/xacro">
+<?xml version="1.0" encoding="utf-8"?>
+<robot name="sensor_asus_xtion_pro" xmlns:xacro="http://www.ros.org/wiki/xacro"> <!-- ASUS Xtion PRO LIVE -->
   <xacro:include filename="$(find turtlex_description)/urdf/asus_xtion_pro_gazebo.urdf.xacro"/>
   <!-- Xacro properties -->
-  <!--<xacro:property name="cam_px" value="-0.087" />-->
-  <!--<xacro:property name="cam_py" value="0.0205"/>-->
-  <!--<xacro:property name="cam_pz" value="0.2870" />-->
   <xacro:property name="cam_px" value="0.174" />
   <xacro:property name="cam_py" value="0.0225"/>
@@ -45,5 +42,4 @@
         <origin xyz="0.0 0.0 0.0" rpy="0 0 0" />
         <geometry>
-        <!--<box size="0.0730 0.2760 0.0720"/>-->
         <box size="0.039 0.19 0.032"/>
       </geometry>
@@ -73,5 +69,4 @@
     <!-- Asus mount -->
     <joint name="mount_asus_xtion_pro_joint" type="fixed">
-      <!--<origin xyz="-0.1024 0.0 0.272" rpy="0 0 0"/>-->
       <origin xyz="0.155 0.0 0.0826" rpy="0 0 0"/>
       <parent link="${parent}"/>
@@ -88,5 +83,4 @@
         <origin xyz="0.0 0.0 0.0" rpy="0 0 0" />
         <geometry>
-        <!--<box size="0.0330 0.2760 0.0120"/>-->
         <box size="0.0330 0.2260 0.0120"/>
       </geometry>

File: turtlex/turtlex_description/urdf/asus_xtion_pro_gazebo.urdf.xacro (robot description, xacro)
@@ -1,5 +1,5 @@
-<?xml version="1.0" encoding="utf-8"?> <!-- NOTA BENE: questa e la asus xtion pro LIVE (quella non live non ha rgb) -->
+<?xml version="1.0" encoding="utf-8"?>
 <robot name="asus_xtion_pro_gazebo" xmlns:xacro="http://www.ros.org/wiki/xacro">
-  <!-- ASUS Xtion PRO for simulation -->
+  <!-- ASUS Xtion PRO LIVE for simulation -->
   <xacro:macro name="asus_xtion_pro_sim_3dsensor">
     <gazebo reference="camera_link">
@@ -19,8 +19,8 @@
           </clip>
         </camera>
-        <plugin name="camera_plugin" filename="libgazebo_ros_openni_kinect.so"> <!-- rinomina come asus_xtion_pro_camera_controller ? -->
+        <plugin name="asus_xtion_pro_camera_controller" filename="libgazebo_ros_openni_kinect.so">
           <cameraName>camera</cameraName>
           <alwaysOn>true</alwaysOn>
-          <updateRate>10</updateRate> <!-- <updateRate>0</updateRate> -->
+          <updateRate>10</updateRate>
           <imageTopicName>rgb/image_raw</imageTopicName>
           <depthImageTopicName>depth/image_raw</depthImageTopicName>

File: turtlex/turtlex_description/urdf/common_properties.urdf.xacro (robot description, xacro)
@@ -2,5 +2,5 @@
 <!--
   Various useful properties such as constants and materials
- -->
+-->
 <robot name="xacro_properties" xmlns:xacro="http://www.ros.org/wiki/xacro">
   <xacro:property name="M_PI" value="3.1415926535897931" />

File: turtlex/turtlex_description/urdf/hexagons.urdf.xacro (robot description, xacro)
@@ -2,5 +2,5 @@
 <!--
   Hexagon stacks
- -->
+-->
 <robot name="stack_hexagons" xmlns:xacro="http://ros.org/wiki/xacro">
   <!-- Xacro properties -->

File: turtlex/turtlex_description/urdf/kobuki.urdf.xacro (robot description, xacro)
@@ -5,7 +5,6 @@
   See kobuki_standalone.urdf.xacro for a standalone urdf to be tested with
       turtlex_description/launch/view_model.launch
- -->
+-->
 <robot name="kobuki" xmlns:xacro="http://www.ros.org/wiki/xacro">
-  <!--<xacro:include filename="$(find turtlex_description)/urdf/common_properties.urdf.xacro"/>-->
   <xacro:include filename="$(find turtlex_description)/urdf/kobuki_gazebo.urdf.xacro"/>
   <!-- Kobuki -->
@@ -20,5 +19,5 @@
        axis, set the z-distance from the base_footprint
        to 0.352.
-      -->
+    -->
     <joint name="base_joint" type="fixed">
       <origin xyz="0 0 0.0102" rpy="0 0 0" />
@@ -29,5 +28,4 @@
       <visual>
         <geometry>
-          <!-- new mesh -->
           <mesh filename="package://turtlex_description/meshes/main_body.dae" />
         </geometry>
@@ -209,7 +207,5 @@
     </link>
     <joint name="laser_sensor_joint" type="fixed">
-    	<!--<origin xyz="0.0 0.0 0.435" rpy="0 0 0"/>-->
       <origin xyz="0.114 0.0 0.038" rpy="0 0 0"/>
-    	<!--<parent link="base_link"/>-->
       <parent link="plate_bottom_link"/>
     	<child link="laser_sensor_link"/>
@@ -224,5 +220,4 @@
 		    <origin xyz="0 0 0" rpy="0 0 0"/>
 		    <geometry>
-			    <!--<box size="0.1 0.1 0.1"/>-->
           <box size="0.05 0.05 0.07"/>
 		    </geometry>

File: turtlex/turtlex_description/urdf/kobuki_gazebo.urdf.xacro (robot description, xacro)
@@ -56,6 +56,36 @@
 	            <samples>50</samples>
 	            <resolution>1.0</resolution>
-	            <min_angle>-0.0436</min_angle>  <!-- -2.5 degree -->
-	            <max_angle>0.0436</max_angle> <!-- 2.5 degree -->
+	            <min_angle>-0.0436</min_angle>  <!-- -2.5 degrees -->
+	            <max_angle>0.0436</max_angle> <!-- 2.5 degrees -->
+	          </horizontal>
+<!--            Can't use vertical rays until this bug is resolved: -->
+<!--            https://bitbucket.org/osrf/gazebo/issue/509/vertical-sensor-doesnt-works -->
+<!-- 	          <vertical> -->
+<!-- 	            <samples>50</samples> -->
+<!-- 	            <resolution>1.0</resolution> -->
+<!-- 	            <min_angle>-0.0436</min_angle>  -2.5 degrees -->
+<!-- 	            <max_angle>0.0436</max_angle> 2.5 degrees -->
+<!-- 	          </vertical> -->
+	        </scan>
+	        <range>
+	          <min>0.01</min>
+	          <max>0.15</max>
+	          <resolution>1.0</resolution>
+	        </range>
+	      </ray>
+	    </sensor>
+	  </gazebo>
+	  <gazebo reference="cliff_sensor_right_link">
+	    <sensor type="ray" name="cliff_sensor_right">
+	      <always_on>true</always_on>
+	      <update_rate>50</update_rate>
+	      <visualize>true</visualize>
+	      <ray>
+	        <scan>
+	          <horizontal>
+	            <samples>50</samples>
+	            <resolution>1.0</resolution>
+	            <min_angle>-0.0436</min_angle> <!-- -2.5 degrees -->
+	            <max_angle>0.0436</max_angle> <!-- 2.5 degrees -->
 	          </horizontal>
 <!--            Can't use vertical rays until this bug is resolved: -->
@@ -76,6 +106,6 @@
 	    </sensor>
 	  </gazebo>
-	  <gazebo reference="cliff_sensor_right_link">
-	    <sensor type="ray" name="cliff_sensor_right">
+	  <gazebo reference="cliff_sensor_front_link">
+	    <sensor type="ray" name="cliff_sensor_front">
 	      <always_on>true</always_on>
 	      <update_rate>50</update_rate>
@@ -86,36 +116,6 @@
 	            <samples>50</samples>
 	            <resolution>1.0</resolution>
-	            <min_angle>-0.0436</min_angle>  <!-- -2.5 degree -->
-	            <max_angle>0.0436</max_angle> <!-- 2.5 degree -->
-	          </horizontal>
-<!--            Can't use vertical rays until this bug is resolved: -->
-<!--            https://bitbucket.org/osrf/gazebo/issue/509/vertical-sensor-doesnt-works -->
-<!-- 	          <vertical> -->
-<!-- 	            <samples>50</samples> -->
-<!-- 	            <resolution>1.0</resolution> -->
-<!-- 	            <min_angle>-0.0436</min_angle>  -2.5 degree -->
-<!-- 	            <max_angle>0.0436</max_angle> 2.5 degree -->
-<!-- 	          </vertical> -->
-	        </scan>
-	        <range>
-	          <min>0.01</min>
-	          <max>0.15</max>
-	          <resolution>1.0</resolution>
-	        </range>
-	      </ray>
-	    </sensor>
-	  </gazebo>
-	  <gazebo reference="cliff_sensor_front_link">
-	    <sensor type="ray" name="cliff_sensor_front">
-	      <always_on>true</always_on>
-	      <update_rate>50</update_rate>
-	      <visualize>true</visualize>
-	      <ray>
-	        <scan>
-	          <horizontal>
-	            <samples>50</samples>
-	            <resolution>1.0</resolution>
-	            <min_angle>-0.0436</min_angle>  <!-- -2.5 degree -->
-	            <max_angle>0.0436</max_angle> <!-- 2.5 degree -->
+	            <min_angle>-0.0436</min_angle> <!-- -2.5 degrees -->
+	            <max_angle>0.0436</max_angle> <!-- 2.5 degrees -->
 	          </horizontal>
 <!-- 	          Can't use vertical rays until this bug is resolved: -->
@@ -124,6 +124,6 @@
 <!-- 	            <samples>50</samples> -->
 <!-- 	            <resolution>1.0</resolution> -->
-<!-- 	            <min_angle>-0.0436</min_angle>  -2.5 degree -->
-<!-- 	            <max_angle>0.0436</max_angle> 2.5 degree -->
+<!-- 	            <min_angle>-0.0436</min_angle>  -2.5 degrees -->
+<!-- 	            <max_angle>0.0436</max_angle> 2.5 degrees -->
 <!-- 	          </vertical> -->
 	        </scan>
@@ -163,12 +163,11 @@
       <plugin name="differential_drive_controller" filename="libgazebo_ros_diff_drive.so">
 	    <alwaysOn>true</alwaysOn>
-	    <updateRate>30</updateRate>	<!--<updateRate>20</updateRate>-->
+	    <updateRate>30</updateRate>
 	    <leftJoint>wheel_left_joint</leftJoint>
     	<rightJoint>wheel_right_joint</rightJoint>
 	    <wheelSeparation>.230</wheelSeparation>
 	    <wheelDiameter>0.070</wheelDiameter>
-	    <!--<torque>1.0</torque>-->
-		<wheelAcceleration>1</wheelAcceleration> <!--<wheelAcceleration>0</wheelAcceleration>-->
-		<wheelTorque>10</wheelTorque> <!--<wheelTorque>5</wheelTorque>-->
+		<wheelAcceleration>1</wheelAcceleration>
+		<wheelTorque>10</wheelTorque>
 	    <commandTopic>cmd_vel</commandTopic>
 	    <odometryTopic>odom</odometryTopic>
@@ -180,5 +179,5 @@
 		<publishWheelJointState>true</publishWheelJointState>
 		<robotBaseFrame>base_footprint</robotBaseFrame>
-	    <legacyMode>false</legacyMode> <!--<legacyMode>true</legacyMode>-->
+	    <legacyMode>false</legacyMode>
 		<rosDebugLevel>na</rosDebugLevel>
 	  </plugin>
@@ -215,21 +214,4 @@
 		</sensor>
 	</gazebo>
-          <!--gazebo>
-	    <plugin name="kobuki_controller" filename="libgazebo_ros_kobuki.so">
-	      <publish_tf>1</publish_tf>
-	      <left_wheel_joint_name>wheel_left_joint</left_wheel_joint_name>
-	      <right_wheel_joint_name>wheel_right_joint</right_wheel_joint_name>
-	      <wheel_separation>.230</wheel_separation>
-	      <wheel_diameter>0.070</wheel_diameter>
-	      <torque>1.0</torque>
-	      <velocity_command_timeout>0.6</velocity_command_timeout>
-	      <cliff_sensor_left_name>cliff_sensor_left</cliff_sensor_left_name>
-	      <cliff_sensor_center_name>cliff_sensor_front</cliff_sensor_center_name>
-	      <cliff_sensor_right_name>cliff_sensor_right</cliff_sensor_right_name>
-	      <cliff_detection_threshold>0.04</cliff_detection_threshold>
-	      <bumper_name>bumpers</bumper_name>
-        <imu_name>imu</imu_name>
-	    </plugin>
-	  </gazebo-->
   </xacro:macro>
 </robot>
