Commit message: Mostly comment removals

File: turtlex/turtlex_description/urdf/widowx.urdf.xacro (robot description, xacro)
@@ -2,5 +2,4 @@
 <robot xmlns:xacro="http://ros.org/wiki/xacro">
    <xacro:property name="M_SCALE" value="0.001"/>
-   <!--<xacro:include filename="$(find turtlex_description)/urdf/common_properties.urdf.xacro" />-->
    <xacro:include filename="$(find turtlex_description)/urdf/widowx_gazebo.urdf.xacro"/>
    <!--link name="plate_top_link"/-->
@@ -142,16 +141,13 @@
          <child link="shoulder_link" />
          <axis xyz="0 0 1" />
-         <!--<limit lower="-2.617" upper="2.617" effort="6" velocity="0.785" />-->
-         <limit lower="-2.617" upper="2.617" effort="50" velocity="0.785" /> <!--era 10000-->
+         <limit lower="-2.617" upper="2.617" effort="50" velocity="0.785" />
          <dynamics friction="0.1"/>
       </joint>
       <joint name="joint_2" type="revolute">
-         <!--origin xyz="0.04825 0 0.14203" rpy="0 0 0" /-->
          <origin xyz="0 0 0" rpy="0 0 0" />
          <parent link="shoulder_link" />
          <child link="biceps_link" />
          <axis xyz="0 1 0" />
-         <!--<limit lower="-1.571" upper="1.571" effort="6" velocity="1.571" />-->
-         <limit lower="-1.571" upper="1.571" effort="50" velocity="1.571" /> <!--era 10000-->
+         <limit lower="-1.571" upper="1.571" effort="50" velocity="1.571" />
          <dynamics friction="0.1"/>
       </joint>
@@ -161,6 +157,5 @@
          <child link="forearm_link" />
          <axis xyz="0 1 0" />
-         <!--<limit lower="-1.571" upper="1.571" effort="6" velocity="1.571" />-->
-         <limit lower="-1.571" upper="1.571" effort="50" velocity="1.571" /> <!--era 10000-->
+         <limit lower="-1.571" upper="1.571" effort="50" velocity="1.571" />
          <dynamics friction="0.1"/>
       </joint>
@@ -170,6 +165,5 @@
          <child link="wrist_1_link" />
          <axis xyz="0 1 0" />
-         <!--<limit lower="-1.745" upper="1.745" effort="6" velocity="1.571" />-->
-         <limit lower="-1.745" upper="1.745" effort="50" velocity="1.571" /> <!--era 10000-->
+         <limit lower="-1.745" upper="1.745" effort="50" velocity="1.571" />
          <dynamics friction="0.1"/>
       </joint>
@@ -179,98 +173,94 @@
          <child link="wrist_2_link" />
          <axis xyz="0 0 1" />
-         <!--<limit lower="-2.617" upper="2.617" effort="6" velocity="1.571" />-->
-         <limit lower="-2.617" upper="2.617" effort="50" velocity="1.571" /> <!--era 10000-->
-         <dynamics friction="0.1"/>
-      </joint>
-            <!-- Gripper -->
-            <!--<xacro:include filename="$(find turtlex_description)/urdf/widowx_gripper.xacro"/>-->
-            <link name="gripper_rail_link">
-            <visual>
-               <origin xyz="0 0 0" rpy="0 0 1.57" />
-               <geometry>
-                  <mesh filename="package://turtlex_description/meshes/arm/gripper_rail_link.stl"/>
-               </geometry>
-               <xacro:material_black />
-            </visual>
-            <collision>
-               <origin xyz="0 0 0" rpy="0 0 1.57" />
-               <geometry>
-                  <mesh filename="package://turtlex_description/meshes/arm/gripper_rail_link.stl"/>
-               </geometry>
-            </collision>
-            <inertial>
-               <origin xyz="0 0 0" rpy="0 0 0" />
-               <mass value="0.001" />
-               <inertia ixx="0.001" iyy="0.001" izz="0.001" ixy="0" ixz="0" iyz="0" />
-            </inertial>
-         </link>
-         <link name="gripper_1_link">
-            <visual>
-               <origin xyz="0 -0.0007 0" rpy="0 0 1.57" />
-               <geometry>
-                  <mesh filename="package://turtlex_description/meshes/arm/gripper_hand_fixed_link.stl"/>
-               </geometry>
-               <xacro:material_black />
-            </visual>
-            <collision>
-               <origin xyz="0 -0.0007 0" rpy="0 0 1.57" />
-               <geometry>
-                  <mesh filename="package://turtlex_description/meshes/arm/gripper_hand_fixed_link.stl"/>
-               </geometry>
-            </collision>
-            <inertial>
-               <origin xyz="0 0 0" rpy="0 0 0" />
-               <mass value="0.016246" />
-               <inertia ixx="0.0000047310" iyy="0.0000015506" izz="0.0000037467" ixy="0.0000004560" ixz="0.0000000000" iyz="0.0000000000" />
-            </inertial>
-         </link>
-         <link name="gripper_2_link">
-            <visual>
-               <origin xyz="0 0.0007 0" rpy="0 0 -1.57" />
-               <geometry>
-                  <mesh filename="package://turtlex_description/meshes/arm/gripper_hand_fixed_link.stl"/>
-               </geometry>
-               <xacro:material_black />
-            </visual>
-            <collision>
-               <origin xyz="0 0.0007 0" rpy="0 0 -1.57" />
-               <geometry>
-                  <mesh filename="package://turtlex_description/meshes/arm/gripper_hand_fixed_link.stl"/>
-               </geometry>
-            </collision>
-            <inertial>
-               <origin xyz="0 0 0" rpy="0 0 0" />
-               <mass value="0.016246" />
-               <inertia ixx="0.0000047310" iyy="0.0000015506" izz="0.0000037467" ixy="0.0000004560" ixz="0.0000000000" iyz="0.0000000000" />
-            </inertial>
-         </link>
-         <joint name="joint_6" type="fixed">
-            <origin xyz = "0 0 ${M_SCALE*43}" rpy="0 0 0" />
-            <parent link="wrist_2_link" />
-            <child link="gripper_rail_link" />
-            <axis xyz="0 0 1" />
-         </joint>
-         <joint name="gripper_prismatic_joint_1" type="prismatic">
-            <origin xyz="0 0 0" rpy="0 0 0" />
-            <parent link="gripper_rail_link" />
-            <child link="gripper_1_link" />
-            <axis xyz="0 -1 0" />
-            <!--<limit lower="0.002" upper="0.031" effort="6" velocity="0.5" />--> <!-- lower="0" upper="0.027"  ? -->
-            <limit lower="0.002" upper="0.031" effort="50" velocity="0.5" /> <!--era 10000-->
-            <dynamics friction="0.1"/>
-         </joint>
-         <joint name="gripper_prismatic_joint_2" type="prismatic">
-            <origin xyz="0 0 0" rpy="0 0 0" />
-            <parent link="gripper_rail_link" />
-            <child link="gripper_2_link" />
-            <!--<mimic joint="gripper_prismatic_joint_1" multiplier="-1" offset="0"/>-->
-            <axis xyz="0 1 0" />
-            <!--<limit lower="0.002" upper="0.031" effort="6" velocity="0.5" />--> <!-- lower="0" upper="0.027"  ? -->
-            <limit lower="0.002" upper="0.031" effort="50" velocity="0.5" /> <!--era 10000-->
-            <dynamics friction="0.1"/>
-         </joint>
-         <!--<xacro:mimic_joint_plugin_gazebo name_prefix="gripper_prismatic_joint_2"
-         parent_joint="gripper_prismatic_joint_1" mimic_joint="gripper_prismatic_joint_2"
-         has_pid="true" multiplier="-1.0" max_effort="6" />-->
+         <limit lower="-2.617" upper="2.617" effort="50" velocity="1.571" />
+         <dynamics friction="0.1"/>
+      </joint>
+      <!-- Gripper -->
+      <link name="gripper_rail_link">
+         <visual>
+            <origin xyz="0 0 0" rpy="0 0 1.57" />
+            <geometry>
+               <mesh filename="package://turtlex_description/meshes/arm/gripper_rail_link.stl"/>
+            </geometry>
+            <xacro:material_black />
+         </visual>
+         <collision>
+            <origin xyz="0 0 0" rpy="0 0 1.57" />
+            <geometry>
+               <mesh filename="package://turtlex_description/meshes/arm/gripper_rail_link.stl"/>
+            </geometry>
+         </collision>
+         <inertial>
+            <origin xyz="0 0 0" rpy="0 0 0" />
+            <mass value="0.001" />
+            <inertia ixx="0.001" iyy="0.001" izz="0.001" ixy="0" ixz="0" iyz="0" />
+         </inertial>
+      </link>
+      <link name="gripper_1_link">
+         <visual>
+            <origin xyz="0 -0.0007 0" rpy="0 0 1.57" />
+            <geometry>
+               <mesh filename="package://turtlex_description/meshes/arm/gripper_hand_fixed_link.stl"/>
+            </geometry>
+            <xacro:material_black />
+         </visual>
+         <collision>
+            <origin xyz="0 -0.0007 0" rpy="0 0 1.57" />
+            <geometry>
+               <mesh filename="package://turtlex_description/meshes/arm/gripper_hand_fixed_link.stl"/>
+            </geometry>
+         </collision>
+         <inertial>
+            <origin xyz="0 0 0" rpy="0 0 0" />
+            <mass value="0.016246" />
+            <inertia ixx="0.0000047310" iyy="0.0000015506" izz="0.0000037467" ixy="0.0000004560" ixz="0.0000000000" iyz="0.0000000000" />
+         </inertial>
+      </link>
+      <link name="gripper_2_link">
+         <visual>
+            <origin xyz="0 0.0007 0" rpy="0 0 -1.57" />
+            <geometry>
+               <mesh filename="package://turtlex_description/meshes/arm/gripper_hand_fixed_link.stl"/>
+            </geometry>
+            <xacro:material_black />
+         </visual>
+         <collision>
+            <origin xyz="0 0.0007 0" rpy="0 0 -1.57" />
+            <geometry>
+               <mesh filename="package://turtlex_description/meshes/arm/gripper_hand_fixed_link.stl"/>
+            </geometry>
+         </collision>
+         <inertial>
+            <origin xyz="0 0 0" rpy="0 0 0" />
+            <mass value="0.016246" />
+            <inertia ixx="0.0000047310" iyy="0.0000015506" izz="0.0000037467" ixy="0.0000004560" ixz="0.0000000000" iyz="0.0000000000" />
+         </inertial>
+      </link>
+      <joint name="joint_6" type="fixed">
+         <origin xyz = "0 0 ${M_SCALE*43}" rpy="0 0 0" />
+         <parent link="wrist_2_link" />
+         <child link="gripper_rail_link" />
+         <axis xyz="0 0 1" />
+      </joint>
+      <joint name="gripper_prismatic_joint_1" type="prismatic">
+         <origin xyz="0 0 0" rpy="0 0 0" />
+         <parent link="gripper_rail_link" />
+         <child link="gripper_1_link" />
+         <axis xyz="0 -1 0" />
+         <limit lower="0.002" upper="0.031" effort="50" velocity="0.5" />
+         <dynamics friction="0.1"/>
+      </joint>
+      <joint name="gripper_prismatic_joint_2" type="prismatic">
+         <origin xyz="0 0 0" rpy="0 0 0" />
+         <parent link="gripper_rail_link" />
+         <child link="gripper_2_link" />
+         <!--<mimic joint="gripper_prismatic_joint_1" multiplier="-1" offset="0"/>-->
+         <axis xyz="0 1 0" />
+         <limit lower="0.002" upper="0.031" effort="50" velocity="0.5" />
+         <dynamics friction="0.1"/>
+      </joint>
+      <!--<xacro:mimic_joint_plugin_gazebo name_prefix="gripper_prismatic_joint_2"
+      parent_joint="gripper_prismatic_joint_1" mimic_joint="gripper_prismatic_joint_2"
+      has_pid="true" multiplier="-1.0" max_effort="6" />-->
    </xacro:macro>
   <transmission name="tran1">

File: turtlex/turtlex_description/urdf/widowx_gazebo.urdf.xacro (robot description, xacro)
@@ -5,27 +5,11 @@
   <gazebo>
     <plugin name="gazebo_ros_control" filename="libgazebo_ros_control.so">
-      <!--<robotNamespace>/turtlex</robotNamespace>-->
       <robotSimType>gazebo_ros_control/DefaultRobotHWSim</robotSimType>
     </plugin>
   </gazebo>
-<!--
-    potrebbe essere che qui i gazebo reference siano del tipo:
-    <kp>1000000.0</kp>
-    <kd>100.0</kd>
-    <mu1>1.5</mu1>
-    <mu2>1.5</mu2>
-    <fdir1>1 0 0</fdir1>
-    <maxVel>1.0</maxVel>
-    <minDepth>0.002</minDepth>
--->
-<!--
-  mu1 mu2:
-  https://answers.gazebosim.org/question/22301/friction-parameters-mu1-and-mu2-in-gazebo-reference-tag-wrong-description-in-tutorial/
--->
   <gazebo reference="arm_base_link">
     <mu1>0.2</mu1>
     <mu2>0.2</mu2>
     <material>Gazebo/DarkGrey</material>
-    <!--<dampingFactor>0.1</dampingFactor>-->
   </gazebo>
   <gazebo reference="shoulder_link">
@@ -33,5 +17,4 @@
     <mu2>0.2</mu2>
     <material>Gazebo/Grey</material>
-    <!--<dampingFactor>0.1</dampingFactor>-->
   </gazebo>
   <gazebo reference="biceps_link">
@@ -39,5 +22,4 @@
     <mu2>0.2</mu2>
     <material>Gazebo/DarkGrey</material>
-    <!--<dampingFactor>0.1</dampingFactor>-->
   </gazebo>
   <gazebo reference="forearm_link">
@@ -45,5 +27,4 @@
     <mu2>0.2</mu2>
     <material>Gazebo/Grey</material>
-    <!--<dampingFactor>0.1</dampingFactor>-->
   </gazebo>
   <gazebo reference="wrist_1_link">
@@ -51,5 +32,4 @@
     <mu2>0.2</mu2>
     <material>Gazebo/DarkGrey</material>
-    <!--<dampingFactor>0.1</dampingFactor>-->
   </gazebo>
   <gazebo reference="wrist_2_link">
@@ -57,5 +37,4 @@
     <mu2>0.2</mu2>
     <material>Gazebo/DarkGrey</material>
-    <!--<dampingFactor>0.1</dampingFactor>-->
   </gazebo>
   <gazebo reference="gripper_rail_link">
@@ -63,14 +42,6 @@
     <mu2>0.2</mu2>
     <material>Gazebo/Grey</material>
-    <!--<dampingFactor>0.1</dampingFactor>-->
   </gazebo>
-  <!--
-    forse conviene mettere a 10 mu1 e mu2 (friction) per i gripper links (o forse mu2 > mu1), vedi qui:
-    https://answers.gazebosim.org/question/22301/friction-parameters-mu1-and-mu2-in-gazebo-reference-tag-wrong-description-in-tutorial/
-    https://answers.gazebosim.org//question/22303/object-slips-from-gripper-fingers-when-grasping-in-simulation/
-  -->
   <gazebo reference="gripper_1_link">
-    <!--<mu1>0.2</mu1>-->
-    <!--<mu2>0.2</mu2>-->
     <kp>1000000.0</kp>
     <kd>100.0</kd>
@@ -80,9 +51,6 @@
     <minDepth>0.001</minDepth>
     <material>Gazebo/Grey</material>
-    <!--<dampingFactor>0.1</dampingFactor>-->
   </gazebo>
   <gazebo reference="gripper_2_link">
-    <!--<mu1>0.2</mu1>-->
-    <!--<mu2>0.2</mu2>-->
     <kp>1000000.0</kp>
     <kd>100.0</kd>
@@ -92,5 +60,4 @@
     <minDepth>0.001</minDepth>
     <material>Gazebo/Grey</material>
-    <!--<dampingFactor>0.1</dampingFactor>-->
   </gazebo>
   </xacro:macro>
