Commit message: Mostly done with cleanups; solved dropbox abs path issue: (see descr.)
now the turtlex_gazebo package is machine-independent

File: turtlex/turtlex_description/urdf/common_properties.urdf.xacro (robot description, xacro)
@@ -55,4 +55,5 @@
     </material>
   </xacro:property>
+  <!-- Colors definition -->
   <!-- RAL 1021 -->
 	<xacro:property name="color_yellow"   value="0.96 0.76 0.13 1.0" />
@@ -61,5 +62,4 @@
 	<!-- RAL 7024 -->
 	<xacro:property name="color_grey"     value="0.34 0.35 0.36 1.0" />
-	<!-- approximations -->
 	<xacro:property name="color_black"    value="0.15 0.15 0.15 1.0" />
 	<xacro:property name="color_greyish"  value="0.75 0.75 0.75 1.0" />

File: turtlex/turtlex_description/urdf/kobuki.urdf.xacro (robot description, xacro)
@@ -48,5 +48,5 @@
              iyy = 1/12 * m * (3 * r^2 + h^2)
              izz = 1/2 * m * r^2
-          -->
+        -->
         <inertia ixx="0.019995" ixy="0.0" ixz="0.0"
                  iyy="0.019995" iyz="0.0"

File: turtlex/turtlex_description/urdf/widowx.urdf.xacro (robot description, xacro)
@@ -3,11 +3,6 @@
    <xacro:property name="M_SCALE" value="0.001"/>
    <xacro:include filename="$(find turtlex_description)/urdf/widowx_gazebo.urdf.xacro"/>
-   <!--link name="plate_top_link"/-->
-   <!--joint name="fixed" type="fixed">
-      <parent link="plate_top_link" />
-      <child link="ph_base_link" />
-   </joint-->
    <xacro:macro name="widowx_arm" params="parent *origin">
-      <!-- links -->
+      <!-- Links -->
       <link name="arm_base_link">
          <visual>
@@ -54,12 +49,12 @@
             <origin xyz="0 0 0" rpy="0 0 0" />
             <geometry>
-               <mesh filename="package://turtlex_description/meshes/arm/biceps_link.new.stl" />
-            </geometry>
-            <xacro:material_black />
-         </visual>
-         <collision>
-            <origin xyz="0 0 0" rpy="0 0 0" />
-            <geometry>
-               <mesh filename="package://turtlex_description/meshes/arm/biceps_link.new.stl" />
+               <mesh filename="package://turtlex_description/meshes/arm/biceps_link.stl" />
+            </geometry>
+            <xacro:material_black />
+         </visual>
+         <collision>
+            <origin xyz="0 0 0" rpy="0 0 0" />
+            <geometry>
+               <mesh filename="package://turtlex_description/meshes/arm/biceps_link.stl" />
             </geometry>
          </collision>
@@ -74,5 +69,5 @@
             <origin xyz="0 0 0" rpy="0 0 0" />
             <geometry>
-               <mesh filename="package://turtlex_description/meshes/arm/forearm_link.new.stl"/>
+               <mesh filename="package://turtlex_description/meshes/arm/forearm_link.stl"/>
             </geometry>
            <xacro:material_black />
@@ -81,5 +76,5 @@
             <origin xyz="0 0 0" rpy="0 0 0" />
             <geometry>
-               <mesh filename="package://turtlex_description/meshes/arm/forearm_link.new.stl"/>
+               <mesh filename="package://turtlex_description/meshes/arm/forearm_link.stl"/>
             </geometry>
          </collision>
@@ -114,12 +109,12 @@
             <origin xyz="0 0 0" rpy="0 0 0" />
             <geometry>
-               <mesh filename="package://turtlex_description/meshes/arm/wrist_2_link.new.stl"/>
-            </geometry>
-            <xacro:material_black />
-         </visual>
-         <collision>
-            <origin xyz="0 0 0" rpy="0 0 0" />
-            <geometry>
-               <mesh filename="package://turtlex_description/meshes/arm/wrist_2_link.new.stl"/>
+               <mesh filename="package://turtlex_description/meshes/arm/wrist_2_link.stl"/>
+            </geometry>
+            <xacro:material_black />
+         </visual>
+         <collision>
+            <origin xyz="0 0 0" rpy="0 0 0" />
+            <geometry>
+               <mesh filename="package://turtlex_description/meshes/arm/wrist_2_link.stl"/>
             </geometry>
          </collision>
@@ -130,5 +125,5 @@
          </inertial>
       </link>
-      <!-- joints -->
+      <!-- Joints -->
       <joint name="arm_base_joint" type="fixed">
          <xacro:insert_block name="origin" />
@@ -255,12 +250,8 @@
          <parent link="gripper_rail_link" />
          <child link="gripper_2_link" />
-         <!--<mimic joint="gripper_prismatic_joint_1" multiplier="-1" offset="0"/>-->
          <axis xyz="0 1 0" />
          <limit lower="0.002" upper="0.031" effort="50" velocity="0.5" />
          <dynamics friction="0.1"/>
       </joint>
-      <!--<xacro:mimic_joint_plugin_gazebo name_prefix="gripper_prismatic_joint_2"
-      parent_joint="gripper_prismatic_joint_1" mimic_joint="gripper_prismatic_joint_2"
-      has_pid="true" multiplier="-1.0" max_effort="6" />-->
    </xacro:macro>
   <transmission name="tran1">
@@ -312,5 +303,4 @@
     <type>transmission_interface/SimpleTransmission</type>
     <joint name="gripper_prismatic_joint_1">
-    <!--<joint name="gripper_joint">-->
       <hardwareInterface>hardware_interface/EffortJointInterface</hardwareInterface>
     </joint>
